Commit message: Added Direct Gripper Driver

File: src/megajaw_description/urdf/pidirect.ros2control.xacro (robot description, xacro)
@@ -4,6 +4,7 @@
         <hardware>
             <plugin>megajaw_hardware_direct/MegaJawHardwareDirect</plugin>
-            <param name="left_wheel_pin_a">5</param>
-            <param name="left_wheel_pin_b">6</param>
+            <param name="servo_pin">5</param>
+            <param name="left_wheel_pin_a">6</param>
+            <param name="left_wheel_pin_b">13</param>
             <param name="right_wheel_pin_a">26</param>
             <param name="right_wheel_pin_b">19</param>
@@ -15,4 +16,9 @@
             <command_interface name="velocity" />
         </joint>
+        <joint name="gripper_ef1_base_joint">
+            <command_interface name="position" />
+            <state_interface name="position" />
+            <state_interface name="velocity" />
+        </joint>
     </ros2_control>
 </robot>
