Commit message: added ros2 control

File: src/megajaw_description/urdf/body.xacro (robot description, xacro)
@@ -32,5 +32,5 @@
     </link>
     <joint name="base_footprint_joint" type="fixed">
-        <origin xyz="0 0 ${base_lz / 2}" rpy="0 0 0" />
+        <origin xyz="0 0 ${base_lz / 2 + wheel_radius}" rpy="0 0 0" />
         <parent link="base_footprint" />
         <child link="base_link" />
@@ -54,6 +54,6 @@
     </link>
     <joint name="left_wheel_base_joint" type="continuous">
-        <origin xyz="${wheel_offset_x} -${base_ly / 2 + wheel_length / 2} ${wheel_offset_z}"
-            rpy="${pi/2} 0 0" />
+        <origin xyz="${wheel_offset_x} ${base_ly / 2 + wheel_length / 2} ${wheel_offset_z}"
+            rpy="${-pi/2} 0 0" />
         <parent link="base_link" />
         <child link="left_wheel_link" />
@@ -78,6 +78,6 @@
     </link>
     <joint name="right_wheel_base_joint" type="continuous">
-        <origin xyz="${wheel_offset_x} ${base_ly / 2 + wheel_length / 2} ${wheel_offset_z}"
-            rpy="${pi/2} 0 0" />
+        <origin xyz="${wheel_offset_x} -${base_ly / 2 + wheel_length / 2} ${wheel_offset_z}"
+            rpy="${-pi/2} 0 0" />
         <parent link="base_link" />
         <child link="right_wheel_link" />

Commit message: added gripper urdf

File: src/megajaw_description/urdf/body.xacro (robot description, xacro)
@@ -17,5 +17,15 @@
     <xacro:property name="camera_ly" value="0.025" />
     <xacro:property name="camera_lz" value="0.023" />
-    <xacro:property name="camera_offset_z" value="${-base_lz / 2 + 0.04}" />
+    <xacro:property name="camera_offset_z" value="${-base_lz / 2 + 0.09}" />
+    <xacro:property name="gripper_base_lx" value="0.048" />
+    <xacro:property name="gripper_base_ly" value="0.062" />
+    <xacro:property name="gripper_base_lz" value="0.032" />
+    <xacro:property name="gripper_base_offset_x" value="0.038" />
+    <xacro:property name="gripper_base_mass" value="0.03" />
+    <xacro:property name="gripper_ef_lx" value="0.083" />
+    <xacro:property name="gripper_ef_ly" value="0.008" />
+    <xacro:property name="gripper_ef_lz" value="0.005" />
+    <xacro:property name="gripper_ef_offset_y" value="0.01" />
+    <xacro:property name="gripper_ef_mass" value="0.01" />
     <link name="base_footprint"></link>
     <link name="base_link">
@@ -110,3 +120,77 @@
         <child link="caster_link" />
     </joint>
+    <!-- Gripper -->
+    <link name="gripper_base_link">
+        <visual>
+            <origin xyz="0 0 ${gripper_base_lz / 2}" rpy="0 0 0" />
+            <geometry>
+                <box size="${gripper_base_lx} ${gripper_base_ly} ${gripper_base_lz}" />
+            </geometry>
+            <material name="brown" />
+        </visual>
+        <collision>
+            <origin xyz="0 0 ${gripper_base_lz / 2}" rpy="0 0 0" />
+            <geometry>
+                <box size="${gripper_base_lx} ${gripper_base_ly} ${gripper_base_lz}" />
+            </geometry>
+        </collision>
+        <xacro:box_inertial m="${gripper_base_mass}" lx="${gripper_base_lx}" ly="${gripper_base_ly}"
+            lz="${gripper_base_lz}" o_xyz="0 0 ${gripper_base_lz / 2}" o_rpy="0 0 0" />
+    </link>
+    <joint name="gripper_base_base_joint" type="fixed">
+        <origin xyz="${gripper_base_offset_x + gripper_base_lx / 2} 0 ${-base_lz / 2 + 0.005}"
+            rpy="0 0 0" />
+        <parent link="base_link" />
+        <child link="gripper_base_link" />
+    </joint>
+    <link name="gripper_ef1_link">
+        <visual>
+            <origin xyz="${gripper_ef_lx / 2} 0 0" rpy="0 0 0" />
+            <geometry>
+                <box size="${gripper_ef_lx} ${gripper_ef_ly} ${gripper_ef_lz}" />
+            </geometry>
+            <material name="green" />
+        </visual>
+        <collision>
+            <origin xyz="${gripper_ef_lx / 2} 0 0" rpy="0 0 0" />
+            <geometry>
+                <box size="${gripper_ef_lx} ${gripper_ef_ly} ${gripper_ef_lz}" />
+            </geometry>
+            <material name="green" />
+        </collision>
+        <xacro:box_inertial m="${gripper_ef_mass}" lx="${gripper_ef_lx}" ly="${gripper_ef_ly}"
+            lz="${gripper_ef_lz}" o_xyz="${gripper_ef_lx / 2} 0 0" o_rpy="0 0 0" />
+    </link>
+    <joint name="gripper_ef1_base_joint" type="revolute">
+        <origin xyz="0 ${gripper_ef_offset_y} ${gripper_base_lz}" rpy="0 0 0" />
+        <parent link="gripper_base_link" />
+        <child link="gripper_ef1_link" />
+        <axis xyz="0 0 1" />
+        <limit lower="0" upper="${pi / 2}" effort="100" velocity="1" />
+    </joint>
+    <link name="gripper_ef2_link">
+        <visual>
+            <origin xyz="${gripper_ef_lx / 2} 0 0" rpy="0 0 0" />
+            <geometry>
+                <box size="${gripper_ef_lx} ${gripper_ef_ly} ${gripper_ef_lz}" />
+            </geometry>
+            <material name="green" />
+        </visual>
+        <collision>
+            <origin xyz="${gripper_ef_lx / 2} 0 0" rpy="0 0 0" />
+            <geometry>
+                <box size="${gripper_ef_lx} ${gripper_ef_ly} ${gripper_ef_lz}" />
+            </geometry>
+            <material name="green" />
+        </collision>
+        <xacro:box_inertial m="${gripper_ef_mass}" lx="${gripper_ef_lx}" ly="${gripper_ef_ly}"
+            lz="${gripper_ef_lz}" o_xyz="${gripper_ef_lx / 2} 0 0" o_rpy="0 0 0" />
+    </link>
+    <joint name="gripper_ef2_base_joint" type="revolute">
+        <origin xyz="0 ${-gripper_ef_offset_y} ${gripper_base_lz}" rpy="0 0 0" />
+        <parent link="gripper_base_link" />
+        <child link="gripper_ef2_link" />
+        <axis xyz="0 0 1" />
+        <limit lower="-${pi / 2}" upper="0" effort="100" velocity="1" />
+    </joint>
 </robot>

File: src/megajaw_description/urdf/materials.xacro (robot description, xacro)
@@ -16,3 +16,6 @@
         <color rgba="0.33 0.33 0.33 1.0"/>
     </material>
+    <material name="brown">
+        <color rgba="0.588 0.294 1.0"/>
+    </material>
 </robot>

Commit message: Cahnges Gripper behaviour to use the ros2_control default node, but sends over UART

File: src/megajaw_description/urdf/body.xacro (robot description, xacro)
@@ -167,5 +167,5 @@
         <child link="gripper_ef1_link" />
         <axis xyz="0 0 1" />
-        <limit lower="0" upper="${pi / 2}" effort="100" velocity="1" />
+        <limit lower="0" upper="0.7" effort="1000" velocity="1" />
     </joint>
     <link name="gripper_ef2_link">
@@ -192,5 +192,5 @@
         <child link="gripper_ef2_link" />
         <axis xyz="0 0 1" />
-        <limit lower="-${pi / 2}" upper="0" effort="100" velocity="1" />
+        <limit lower="-0.7" upper="0" effort="1000" velocity="1" />
     </joint>
 </robot>

File: src/megajaw_description/urdf/gz.ros2control.xacro (robot description, xacro)
@@ -20,7 +20,11 @@
         <joint name="gripper_ef1_base_joint">
             <command_interface name="position" />
+            <state_interface name="position" />
+            <state_interface name="velocity" />
         </joint>
         <joint name="gripper_ef2_base_joint">
             <command_interface name="position" />
+            <state_interface name="position" />
+            <state_interface name="velocity" />
         </joint>
     </ros2_control>

Commit message: modified fsm logic to lock first

File: src/megajaw_description/urdf/body.xacro (robot description, xacro)
@@ -20,11 +20,11 @@
     <xacro:property name="gripper_base_lx" value="0.048" />
     <xacro:property name="gripper_base_ly" value="0.062" />
-    <xacro:property name="gripper_base_lz" value="0.032" />
-    <xacro:property name="gripper_base_offset_x" value="0.038" />
     <xacro:property name="gripper_base_mass" value="0.03" />
     <xacro:property name="gripper_ef_lx" value="0.083" />
     <xacro:property name="gripper_ef_ly" value="0.008" />
     <xacro:property name="gripper_ef_lz" value="0.005" />
+    <xacro:property name="gripper_ef_offset_x" value="${base_lx / 2}" />
     <xacro:property name="gripper_ef_offset_y" value="0.01" />
+    <xacro:property name="gripper_ef_offset_z" value="0" />
     <xacro:property name="gripper_ef_mass" value="0.01" />
     <link name="base_footprint"></link>
@@ -120,28 +120,4 @@
         <child link="caster_link" />
     </joint>
-    <!-- Gripper -->
-    <link name="gripper_base_link">
-        <visual>
-            <origin xyz="0 0 ${gripper_base_lz / 2}" rpy="0 0 0" />
-            <geometry>
-                <box size="${gripper_base_lx} ${gripper_base_ly} ${gripper_base_lz}" />
-            </geometry>
-            <material name="brown" />
-        </visual>
-        <collision>
-            <origin xyz="0 0 ${gripper_base_lz / 2}" rpy="0 0 0" />
-            <geometry>
-                <box size="${gripper_base_lx} ${gripper_base_ly} ${gripper_base_lz}" />
-            </geometry>
-        </collision>
-        <xacro:box_inertial m="${gripper_base_mass}" lx="${gripper_base_lx}" ly="${gripper_base_ly}"
-            lz="${gripper_base_lz}" o_xyz="0 0 ${gripper_base_lz / 2}" o_rpy="0 0 0" />
-    </link>
-    <joint name="gripper_base_base_joint" type="fixed">
-        <origin xyz="${gripper_base_offset_x + gripper_base_lx / 2} 0 ${-base_lz / 2 + 0.005}"
-            rpy="0 0 0" />
-        <parent link="base_link" />
-        <child link="gripper_base_link" />
-    </joint>
     <link name="gripper_ef1_link">
         <visual>
@@ -163,6 +139,6 @@
     </link>
     <joint name="gripper_ef1_base_joint" type="revolute">
-        <origin xyz="0 ${gripper_ef_offset_y} ${gripper_base_lz}" rpy="0 0 0" />
-        <parent link="gripper_base_link" />
+        <origin xyz="${gripper_ef_offset_x} ${gripper_ef_offset_y} ${gripper_ef_offset_z}" rpy="0 0 0" />
+        <parent link="base_link" />
         <child link="gripper_ef1_link" />
         <axis xyz="0 0 1" />
@@ -188,6 +164,6 @@
     </link>
     <joint name="gripper_ef2_base_joint" type="revolute">
-        <origin xyz="0 ${-gripper_ef_offset_y} ${gripper_base_lz}" rpy="0 0 0" />
-        <parent link="gripper_base_link" />
+        <origin xyz="${gripper_ef_offset_x} ${-gripper_ef_offset_y} ${gripper_ef_offset_z}" rpy="0 0 0" />
+        <parent link="base_link" />
         <child link="gripper_ef2_link" />
         <axis xyz="0 0 1" />

Commit message: updated to just have a single EF for the gripper, teh other is mimic

File: src/megajaw_description/urdf/body.xacro (robot description, xacro)
@@ -165,4 +165,5 @@
     <joint name="gripper_ef2_base_joint" type="revolute">
         <origin xyz="${gripper_ef_offset_x} ${-gripper_ef_offset_y} ${gripper_ef_offset_z}" rpy="0 0 0" />
+        <mimic joint="gripper_ef1_base_joint" multiplier="-1.0" offset="0.0"/>
         <parent link="base_link" />
         <child link="gripper_ef2_link" />

File: src/megajaw_description/urdf/gz.ros2control.xacro (robot description, xacro)
@@ -23,9 +23,4 @@
             <state_interface name="velocity" />
         </joint>
-        <joint name="gripper_ef2_base_joint">
-            <command_interface name="position" />
-            <state_interface name="position" />
-            <state_interface name="velocity" />
-        </joint>
     </ros2_control>
 </robot>

File: src/megajaw_description/urdf/pidirect.ros2control.xacro (robot description, xacro)
@@ -19,5 +19,4 @@
             <command_interface name="position" />
             <state_interface name="position" />
-            <state_interface name="velocity" />
         </joint>
     </ros2_control>
